File: PCB/jays-hackpad.kicad_pcb (KiCad board)
At the start: 2 copper layers, 85 x 72 mm, 9 parts, among them SW1 SW_Push, SW2 SW_Push, SW3 SW_Push, SW4 SW_Push, SW5 SW_Push, SW6 SW_Push, SW7 RotaryEncoder_Switch, U1 XIAO-RP2040-DIP

Commit message: Forgot a few fixes
Parts:
- Brd1: footprint SSD1306:128x64OLED -> KiCad-SSD1306-0.91-OLED-4pin-128x32:SSD1306-0.91-OLED-4pin-128x32
- moved Brd1 26.3 mm to (142.2, 78.5), turned to 180 degrees
- moved SW7 4.68 mm to (144.7, 69.9)
Routing:
- net Net-(Brd1-SDA): track 43.9 -> 26.6 mm
- net Net-(Brd1-SCL): track 43.7 -> 28.5 mm, vias 0 -> 1
- net GND: track 185.1 -> 198.7 mm
- net Net-(Brd1-VCC): track 20.6 -> 11.5 mm, vias 0 -> 1
- net Net-(U1-GPIO28/ADC2/A2): track 81.6 -> 86.7 mm
- net Net-(U1-GPIO27/ADC1/A1): track 62.5 -> 67.6 mm, vias 1 -> 2
- net Net-(U1-GPIO26/ADC0/A0): track 65.0 -> 70.0 mm
- net Net-(U1-GPIO4/MISO): track 42.5 -> 44.8 mm
