File: PCB/jays-hackpad.kicad_sch (KiCad schematic)
At the start: 9 parts, among them SW1 SW_Push, SW2 SW_Push, SW3 SW_Push, SW4 SW_Push, SW5 SW_Push, SW6 SW_Push, SW7 RotaryEncoder_Switch, U1 XIAO-RP2040-DIP

Commit message: Forgot a few fixes
Parts:
- Brd1: footprint SSD1306:128x64OLED -> KiCad-SSD1306-0.91-OLED-4pin-128x32:SSD1306-0.91-OLED-4pin-128x32
Changed lines of the file:
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@@
-	(wire
-		(pts
-			(xy 31.75 154.94) (xy 33.02 154.94)
-		)
-		(stroke
-			(width 0)
-			(type default)
-		)
-	)
 	(wire
 		(pts
@@
 	(wire
 		(pts
+			(xy 31.75 139.7) (xy 100.33 139.7)
+		)
+		(stroke
+			(width 0)
+			(type default)
+		)
+	)
+	(wire
+		(pts
 			(xy 35.56 64.77) (xy 36.83 64.77)
 		)
@@
 	(wire
 		(pts
-			(xy 31.75 76.2) (xy 31.75 154.94)
-		)
-		(stroke
-			(width 0)
-			(type default)
-		)
-	)
-	(wire
-		(pts
 			(xy 20.32 72.39) (xy 36.83 72.39)
 		)
@@
 	(wire
 		(pts
+			(xy 31.75 76.2) (xy 31.75 139.7)
+		)
+		(stroke
+			(width 0)
+			(type default)
+		)
+	)
+	(wire
+		(pts
 			(xy 96.52 101.6) (xy 100.33 101.6)
 		)
@@
 	(wire
 		(pts
-			(xy 33.02 154.94) (xy 33.02 139.7)
-		)
-		(stroke
-			(width 0)
-			(type default)
-		)
-	)
-	(wire
-		(pts
 			(xy 31.75 76.2) (xy 36.83 76.2)
 		)
@@
 		(pts
 			(xy 25.4 45.72) (xy 20.32 45.72)
-		)
-		(stroke
-			(width 0)
-			(type default)
-		)
-	)
-	(wire
-		(pts
-			(xy 33.02 139.7) (xy 100.33 139.7)
 		)
 		(stroke
@@
 			)
 		)
-		(property "Footprint" "SSD1306:128x64OLED"
+		(property "Footprint" "KiCad-SSD1306-0.91-OLED-4pin-128x32:SSD1306-0.91-OLED-4pin-128x32"
 			(at 111.76 55.88 0)
 			(effects
